File: KiCad/Odometer-Amplifier.kicad_sch (KiCad schematic)
At the start: 17 parts, among them J1 DASH_CONN, J2 SENSE_CONN, Q1 2N3904, U1 UC_LM358

Commit message: Completed README.md, fixed naming
Parts:
- R6: now left out of the parts list
Changed lines of the file:
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@@
     (pin "2")
     (instances
-      (project "STM32-Pomodoro"
+      (project "Odometer-Amplifier"
         (path "/e43dba7a-a14f-4ec4-a129-d7939f06e55a"
           (reference "R2") (unit 1)
@@
     (pin "1")
     (instances
-      (project "STM32-Pomodoro"
+      (project "Odometer-Amplifier"
         (path "/e43dba7a-a14f-4ec4-a129-d7939f06e55a"
           (reference "#PWR017") (unit 1)
@@
     (pin "2")
     (instances
-      (project "STM32-Pomodoro"
+      (project "Odometer-Amplifier"
         (path "/e43dba7a-a14f-4ec4-a129-d7939f06e55a"
           (reference "R7") (unit 1)
@@
     (pin "1")
     (instances
-      (project "STM32-Pomodoro"
+      (project "Odometer-Amplifier"
         (path "/e43dba7a-a14f-4ec4-a129-d7939f06e55a"
           (reference "B1") (unit 1)
@@
     (pin "1")
     (instances
-      (project "STM32-Pomodoro"
+      (project "Odometer-Amplifier"
         (path "/e43dba7a-a14f-4ec4-a129-d7939f06e55a"
           (reference "Q1") (unit 1)
@@
     (pin "2")
     (instances
-      (project "STM32-Pomodoro"
+      (project "Odometer-Amplifier"
         (path "/e43dba7a-a14f-4ec4-a129-d7939f06e55a"
           (reference "C1") (unit 1)
@@
     (pin "1")
     (instances
-      (project "STM32-Pomodoro"
+      (project "Odometer-Amplifier"
         (path "/e43dba7a-a14f-4ec4-a129-d7939f06e55a"
           (reference "#PWR09") (unit 1)
@@
     (pin "5")
     (instances
-      (project "STM32-Pomodoro"
+      (project "Odometer-Amplifier"
         (path "/e43dba7a-a14f-4ec4-a129-d7939f06e55a"
           (reference "U1") (unit 2)
@@
     (pin "1")
     (instances
-      (project "STM32-Pomodoro"
+      (project "Odometer-Amplifier"
         (path "/e43dba7a-a14f-4ec4-a129-d7939f06e55a"
           (reference "R3") (unit 1)
@@
     (pin "1")
     (instances
-      (project "STM32-Pomodoro"
+      (project "Odometer-Amplifier"
         (path "/e43dba7a-a14f-4ec4-a129-d7939f06e55a"
           (reference "#PWR06") (unit 1)
@@
     (pin "1")
     (instances
-      (project "STM32-Pomodoro"
+      (project "Odometer-Amplifier"
         (path "/e43dba7a-a14f-4ec4-a129-d7939f06e55a"
           (reference "R1") (unit 1)
@@
     (pin "1")
     (instances
-      (project "STM32-Pomodoro"
+      (project "Odometer-Amplifier"
         (path "/e43dba7a-a14f-4ec4-a129-d7939f06e55a"
           (reference "R4") (unit 1)
@@
     (pin "2")
     (instances
-      (project "STM32-Pomodoro"
+      (project "Odometer-Amplifier"
         (path "/e43dba7a-a14f-4ec4-a129-d7939f06e55a"
           (reference "L1") (unit 1)
@@
     (pin "1")
     (instances
-      (project "STM32-Pomodoro"
+      (project "Odometer-Amplifier"
         (path "/e43dba7a-a14f-4ec4-a129-d7939f06e55a"
           (reference "#PWR04") (unit 1)
@@
     (pin "1")
     (instances
-      (project "STM32-Pomodoro"
+      (project "Odometer-Amplifier"
         (path "/e43dba7a-a14f-4ec4-a129-d7939f06e55a"
           (reference "#PWR02") (unit 1)
@@
     (pin "1")
     (instances
-      (project "STM32-Pomodoro"
+      (project "Odometer-Amplifier"
         (path "/e43dba7a-a14f-4ec4-a129-d7939f06e55a"
           (reference "#PWR05") (unit 1)
@@
     (pin "2")
     (instances
-      (project "STM32-Pomodoro"
+      (project "Odometer-Amplifier"
         (path "/e43dba7a-a14f-4ec4-a129-d7939f06e55a"
           (reference "C2") (unit 1)
@@
     (pin "1")
     (instances
-      (project "STM32-Pomodoro"
+      (project "Odometer-Amplifier"
         (path "/e43dba7a-a14f-4ec4-a129-d7939f06e55a"
           (reference "#PWR07") (unit 1)
@@
     (pin "1")
     (instances
-      (project "STM32-Pomodoro"
+      (project "Odometer-Amplifier"
         (path "/e43dba7a-a14f-4ec4-a129-d7939f06e55a"
           (reference "#PWR012") (unit 1)
@@
     (pin "1")
     (instances
-      (project "STM32-Pomodoro"
+      (project "Odometer-Amplifier"
         (path "/e43dba7a-a14f-4ec4-a129-d7939f06e55a"
           (reference "V2") (unit 1)
@@
     (pin "1")
     (instances
-      (project "STM32-Pomodoro"
+      (project "Odometer-Amplifier"
         (path "/e43dba7a-a14f-4ec4-a129-d7939f06e55a"
           (reference "#PWR01") (unit 1)
@@
     (pin "1")
     (instances
-      (project "STM32-Pomodoro"
+      (project "Odometer-Amplifier"
         (path "/e43dba7a-a14f-4ec4-a129-d7939f06e55a"
           (reference "#PWR010") (unit 1)
@@
     (pin "5")
     (instances
-      (project "STM32-Pomodoro"
+      (project "Odometer-Amplifier"
         (path "/e43dba7a-a14f-4ec4-a129-d7939f06e55a"
           (reference "U1") (unit 1)
@@
     (pin "1")
     (instances
-      (project "STM32-Pomodoro"
+      (project "Odometer-Amplifier"
         (path "/e43dba7a-a14f-4ec4-a129-d7939f06e55a"
           (reference "#PWR013") (unit 1)
@@
     (pin "1")
     (instances
-      (project "STM32-Pomodoro"
+      (project "Odometer-Amplifier"
         (path "/e43dba7a-a14f-4ec4-a129-d7939f06e55a"
           (reference "#PWR018") (unit 1)
@@
     (pin "1")
     (instances
-      (project "STM32-Pomodoro"
+      (project "Odometer-Amplifier"
         (path "/e43dba7a-a14f-4ec4-a129-d7939f06e55a"
           (reference "R5") (unit 1)
@@
     (pin "1")
     (instances
-      (project "STM32-Pomodoro"
+      (project "Odometer-Amplifier"
         (path "/e43dba7a-a14f-4ec4-a129-d7939f06e55a"
           (reference "#PWR08") (unit 1)
@@
   )
   (symbol (lib_id "enel200_uc_kicad7:UC_R") (at 77.47 154.305 0) (unit 1)
-    (in_bom yes) (on_board yes) (dnp no) (fields_autoplaced)
+    (in_bom no) (on_board yes) (dnp no) (fields_autoplaced)
     (property "Reference" "R6" (at 80.01 153.035 0)
       (effects (font (size 1.27 1.27)) (justify left))
@@
     (pin "1")
     (instances
-      (project "STM32-Pomodoro"
+      (project "Odometer-Amplifier"
         (path "/e43dba7a-a14f-4ec4-a129-d7939f06e55a"
           (reference "R6") (unit 1)
@@
     (pin "1")
     (instances
-      (project "STM32-Pomodoro"
+      (project "Odometer-Amplifier"
         (path "/e43dba7a-a14f-4ec4-a129-d7939f06e55a"
           (reference "#PWR015") (unit 1)
@@
     (pin "3")
     (instances
-      (project "STM32-Pomodoro"
+      (project "Odometer-Amplifier"
         (path "/e43dba7a-a14f-4ec4-a129-d7939f06e55a"
           (reference "J2") (unit 1)
@@
     (pin "1")
     (instances
-      (project "STM32-Pomodoro"
+      (project "Odometer-Amplifier"
         (path "/e43dba7a-a14f-4ec4-a129-d7939f06e55a"
           (reference "#PWR011") (unit 1)
@@
     (pin "1")
     (instances
-      (project "STM32-Pomodoro"
+      (project "Odometer-Amplifier"
         (path "/e43dba7a-a14f-4ec4-a129-d7939f06e55a"
           (reference "#PWR014") (unit 1)
@@
     (pin "1")
     (instances
-      (project "STM32-Pomodoro"
+      (project "Odometer-Amplifier"
         (path "/e43dba7a-a14f-4ec4-a129-d7939f06e55a"
           (reference "#PWR019") (unit 1)
@@
     (pin "1")
     (instances
-      (project "STM32-Pomodoro"
+      (project "Odometer-Amplifier"
         (path "/e43dba7a-a14f-4ec4-a129-d7939f06e55a"
           (reference "#FLG01") (unit 1)
@@
     (pin "1")
     (instances
-      (project "STM32-Pomodoro"
+      (project "Odometer-Amplifier"
         (path "/e43dba7a-a14f-4ec4-a129-d7939f06e55a"
           (reference "#PWR016") (unit 1)
@@
     (pin "1")
     (instances
-      (project "STM32-Pomodoro"
+      (project "Odometer-Amplifier"
         (path "/e43dba7a-a14f-4ec4-a129-d7939f06e55a"
           (reference "#PWR03") (unit 1)
@@
     (pin "3")
     (instances
-      (project "STM32-Pomodoro"
+      (project "Odometer-Amplifier"
         (path "/e43dba7a-a14f-4ec4-a129-d7939f06e55a"
           (reference "J1") (unit 1)
@@
     (pin "1")
     (instances
-      (project "STM32-Pomodoro"
+      (project "Odometer-Amplifier"
         (path "/e43dba7a-a14f-4ec4-a129-d7939f06e55a"
           (reference "C3") (unit 1)

Commit message: Updated schema, readme
Parts:
- added D1: 5.6V, Diode_THT:D_DO-35_SOD27_P2.54mm_Vertical_KathodeUp, symbol enel200_uc_kicad7:UC_D_ZENER
Connections:
- net +BATT: now also D1.1 (K)
- net GND: now also D1.2 (A)
Changed lines of the file:
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@@
   (junction (at 149.225 67.945) (diameter 0) (color 0 0 0 0)
+  )
+  (junction (at 54.61 69.85) (diameter 0) (color 0 0 0 0)
   )
   (junction (at 27.94 144.145) (diameter 0) (color 0 0 0 0)
@@
     )
   )
+  (symbol (lib_id "power:GND") (at 54.61 77.47 0) (unit 1)
+    (in_bom yes) (on_board yes) (dnp no) (fields_autoplaced)
+    (property "Reference" "#PWR020" (at 54.61 83.82 0)
+      (effects (font (size 1.27 1.27)) hide)
+    )
+    (property "Value" "GND" (at 54.61 81.915 0)
+      (effects (font (size 1.27 1.27)))
+    )
+    (property "Footprint" "" (at 54.61 77.47 0)
+      (effects (font (size 1.27 1.27)) hide)
+    )
+    (property "Datasheet" "" (at 54.61 77.47 0)
+      (effects (font (size 1.27 1.27)) hide)
+    )
+    (pin "1")
+    (instances
+      (project "Odometer-Amplifier"
+        (path "/e43dba7a-a14f-4ec4-a129-d7939f06e55a"
+          (reference "#PWR020") (unit 1)
+        )
+      )
+    )
+  )
   (symbol (lib_id "enel200_uc_kicad7:UC_L") (at 62.23 69.85 0) (unit 1)
     (in_bom yes) (on_board yes) (dnp no) (fields_autoplaced)
@@
         )
       )
+    )
+  )
+  (symbol (lib_id "enel200_uc_kicad7:UC_D_ZENER") (at 54.61 73.66 90) (unit 1)
+    (in_bom yes) (on_board yes) (dnp no)
+    (property "Reference" "D1" (at 59.055 73.66 90)
+      (effects (font (size 1.27 1.27)) (justify left))
+    )
+    (property "Value" "5.6V" (at 60.96 75.565 90)
+      (effects (font (size 1.27 1.27)) (justify left))
+    )
+    (property "Footprint" "Diode_THT:D_DO-35_SOD27_P2.54mm_Vertical_KathodeUp" (at 59.69 73.66 0)
+      (effects (font (size 1.524 1.524)) hide)
+    )
+    (property "Datasheet" "" (at 54.61 73.66 0)
+      (effects (font (size 1.524 1.524)))
+    )
+    (pin "1")
+    (pin "2")
+    (instances
+      (project "Odometer-Amplifier"
+        (path "/e43dba7a-a14f-4ec4-a129-d7939f06e55a"
+          (reference "D1") (unit 1)
+        )
+      )
